File: kicad/stm32f042_devboard/stm32f042_devboard.kicad_pcb (KiCad board)
At the start: 2 copper layers, 25.4 x 25.4 mm, 18 parts, among them J1 USB_B_Micro, J2 Conn_01x04, J3 Conn_01x09, J4 Conn_01x03, J5 Conn_01x03, J6 Conn_01x03, SW1 SW_Push, U1 STM32F042F6Px, U2 AMS1117-3.3

Commit message: updated
Parts:
- added C10: 1u, Capacitor_SMD:C_0805_2012Metric_Pad1.15x1.40mm_HandSolder, B.Cu at (145.2, 81.9)
- added C6: 100n, Capacitor_SMD:C_0805_2012Metric_Pad1.15x1.40mm_HandSolder, B.Cu at (147.6, 87.1)
- added C7: 100n, Capacitor_SMD:C_0805_2012Metric_Pad1.15x1.40mm_HandSolder, B.Cu at (147.6, 89.3)
- added C8: 4.7u, Capacitor_SMD:C_0805_2012Metric_Pad1.15x1.40mm_HandSolder, B.Cu at (147.6, 85.0)
- added C9: 10n, Capacitor_SMD:C_0805_2012Metric_Pad1.15x1.40mm_HandSolder, B.Cu at (143.0, 81.9)
- moved R2 4.26 mm to (136.9, 85.3), turned to 180 degrees
- moved C5 2.50 mm to (135.6, 81.5), turned to 270 degrees
- moved D2 1.99 mm to (136.9, 87.5), turned to 180 degrees
Connections:
- J1 pad 4: (no net) -> Net-(J1-Pad4)
- J4 pad 1: (no net) -> /filt_in
- J4 pad 3: (no net) -> /vout_in
- J5 pad 2: (no net) -> /ifsig
- U1 pad 10: (no net) -> /ADC_IN4
- U1 pad 7: (no net) -> /ADC_IN1
Routing:
- net /3.3V: track 75.2 -> 86.7 mm, vias 3 -> 4
- net /GND: track 45.7 -> 54.7 mm
- net Net-(D2-Pad1): track 8.95 -> 5.35 mm
- net Net-(C5-Pad1): track 45.8 -> 43.6 mm, vias 2 -> 4
Other:
- board text added: "1"
- board text added: "3.3V"
- board text added: "5V"
- board text added: "ADC0"
- board text added: "BOOT"
- board text added: "GND"
- board text added: "PA5"
- board text added: "PA6"
- board text added: "PA7"
- board text added: "RX2"
- board text added: "SCL"
- board text added: "SDA"
- board text added: "SWCLK"
- board text added: "SWDIO"
- board text added: "TX2"
- board text added: "stm32f042f_devboard iman_202001.1"
- board text removed: "stm32f042f-devboard iman_202001.01"
